Commit message: revised the fishbot.urdf.xacro in chapter6

File: chapt6/chapt6_ws/src/fishbot_description/urdf/first_robot.urdf.xacro (robot description, xacro)
@@ -7,5 +7,5 @@
                 <origin xyz="0 0 0" rpy="0 0 0" />
                 <geometry>
-                    <cylinder length="${length}" radius="${length}" />
+                    <cylinder length="${length}" radius="${radius}" />
                 </geometry>
                 <material name="blue">

File: chapt6/chapt6_ws/src/fishbot_description/urdf/fishbot/fishbot.urdf.xacro (robot description, xacro)
@@ -26,3 +26,4 @@
     <xacro:include filename="$(find fishbot_description)/urdf/fishbot/plugins/gazebo_sensor_plugin.xacro" />
     <xacro:gazebo_sensor_plugin />
+    <xacro:gazebo_control_plugin />
 </robot>
